File: kicad_docs/SSI2130_VCO.sch (KiCad schematic (older format))
At the start: 8 parts, among them J1 tuning controls, J2 1 v/oct inputs, J3 linear FM input, J4 sync input, J5 PWM inputs, J7 waveform outputs

Commit message: fix error where wires were crossed
Changed lines of the file:
@@
 F7 "raw_pulse_out" O R 6450 2450 50
 F8 "raw_tri_out" O R 6450 2250 50
-F9 "lin_FM_in" I L 4950 3150 50
+F9 "lin_FM_in" I L 4950 3050 50
 F10 "fine_tune_in" I L 4950 2250 50
-F11 "time_rev_in" I L 4950 3050 50
+F11 "time_rev_in" I L 4950 3150 50
 F12 "sync_in" I L 4950 3450 50
 F13 "coarse_tune_in" I L 4950 2150 50
